File: src/Eco_display/RS485.kicad_sch (KiCad schematic)
At the start: 14 parts, among them U19 SSP3485U, U4 TBU-CA065-200-WH, U6 TBU-CA065-200-WH

Commit message: Logo, routing, all files
Parts:
- removed U4, U6: TBU-CA065-200-WH, MACHADA_footprints:TBU-CA065-200-WH, symbol MCD_General:TBU-CA065-200-WH
- added L1, L2: L, Inductor_SMD:L_0402_1005Metric, symbol Device:L
Connections:
- net A: now also L1.2
- net B: now also L2.2
- net at D9.1 (K), R37.2, R38.2: now also L1.1
- net at D9.2 (K), R38.1, R39.2: now also L2.1
Changed lines of the file:
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@@
     (stroke (width 0) (type default))
   )
-  (wire (pts (xy 155.575 102.87) (xy 159.385 102.87))
+  (wire (pts (xy 155.575 102.87) (xy 167.005 102.87))
     (stroke (width 0) (type default))
   )
@@
     (stroke (width 0) (type dash_dot))
   )
-  (wire (pts (xy 183.515 87.63) (xy 188.595 87.63))
+  (wire (pts (xy 174.625 87.63) (xy 188.595 87.63))
     (stroke (width 0) (type default))
   )
@@
     (stroke (width 0) (type default))
   )
-  (wire (pts (xy 150.495 87.63) (xy 159.385 87.63))
+  (wire (pts (xy 150.495 87.63) (xy 167.005 87.63))
     (stroke (width 0) (type default))
   )
@@
     (stroke (width 0) (type default))
   )
-  (wire (pts (xy 183.515 102.87) (xy 207.01 102.87))
+  (wire (pts (xy 174.625 102.87) (xy 207.01 102.87))
     (stroke (width 0) (type default))
   )
@@
         (path "/8b9448db-4b1d-4fc2-a488-03ccb6a18691/342f5a5a-4095-4f7f-8eba-841feace6be3"
           (reference "#PWR011") (unit 1)
+        )
+      )
+    )
+  )
+  (symbol (lib_id "Device:L") (at 170.815 102.87 90) (unit 1)
+    (in_bom yes) (on_board yes) (dnp no)
+    (property "Reference" "L2" (at 170.815 97.155 90)
+      (effects (font (size 1.27 1.27)))
+    )
+    (property "Value" "L" (at 170.815 99.695 90)
+      (effects (font (size 1.27 1.27)))
+    )
+    (property "Footprint" "Inductor_SMD:L_0402_1005Metric" (at 170.815 102.87 0)
+      (effects (font (size 1.27 1.27)) hide)
+    )
+    (property "Datasheet" "~" (at 170.815 102.87 0)
+      (effects (font (size 1.27 1.27)) hide)
+    )
+    (property "MPN" "BLM15HD182SN1D" (at 170.815 104.14 90)
+      (effects (font (size 1.27 1.27)))
+    )
+    (pin "1")
+    (pin "2")
+    (instances
+      (project "Eco_display"
+        (path "/8b9448db-4b1d-4fc2-a488-03ccb6a18691/342f5a5a-4095-4f7f-8eba-841feace6be3"
+          (reference "L2") (unit 1)
         )
       )
@@
     )
   )
-  (symbol (lib_id "MCD_General:TBU-CA065-200-WH") (at 169.545 82.55 0) (unit 1)
-    (in_bom yes) (on_board yes) (dnp no) (fields_autoplaced)
-    (property "Reference" "U4" (at 171.45 81.915 0)
-      (effects (font (size 1.27 1.27)))
-    )
-    (property "Value" "TBU-CA065-200-WH" (at 171.45 84.455 0)
-      (effects (font (size 1.27 1.27)))
-    )
-    (property "Footprint" "MACHADA_footprints:TBU-CA065-200-WH" (at 169.545 83.82 0)
-      (effects (font (size 1.27 1.27)) hide)
-    )
-    (property "Datasheet" "" (at 169.545 83.82 0)
-      (effects (font (size 1.27 1.27)) hide)
-    )
-    (pin "1")
-    (pin "2")
-    (instances
-      (project "Eco_display"
-        (path "/8b9448db-4b1d-4fc2-a488-03ccb6a18691/342f5a5a-4095-4f7f-8eba-841feace6be3"
-          (reference "U4") (unit 1)
-        )
-      )
-      (project "BIM_PCB"
-        (path "/b79ebed7-e146-448b-8dab-0aefb3e182ca/1465f310-1de3-424a-8f4a-a980ed628081"
-          (reference "U4") (unit 1)
-        )
-        (path "/b79ebed7-e146-448b-8dab-0aefb3e182ca/34e5006d-2f61-4d7d-acbf-5a24a5d8c7fc"
-          (reference "U10") (unit 1)
-        )
-        (path "/b79ebed7-e146-448b-8dab-0aefb3e182ca/2e21452f-cdd1-4ce6-a8e8-98e1abc18b72"
-          (reference "U18") (unit 1)
-        )
-      )
-      (project "MAX485"
-        (path "/bc82bdd3-8c90-4895-abd4-de755b621eab"
-          (reference "U13") (unit 1)
-        )
-      )
-      (project "ELIESTER_V2"
-        (path "/efe55700-0211-4481-aa01-7a7eb74def17/d62e2e8a-503b-4c7c-a2bb-b074e6b71fb0"
-          (reference "U13") (unit 1)
-        )
-      )
-    )
-  )
   (symbol (lib_id "Diode:SD05_SOD323") (at 207.01 110.49 90) (unit 1)
     (in_bom yes) (on_board yes) (dnp no) (fields_autoplaced)
@@
         (path "/efe55700-0211-4481-aa01-7a7eb74def17/d62e2e8a-503b-4c7c-a2bb-b074e6b71fb0"
           (reference "#PWR089") (unit 1)
-        )
-      )
-    )
-  )
-  (symbol (lib_id "MCD_General:TBU-CA065-200-WH") (at 169.545 97.79 0) (unit 1)
-    (in_bom yes) (on_board yes) (dnp no) (fields_autoplaced)
-    (property "Reference" "U6" (at 171.45 97.155 0)
-      (effects (font (size 1.27 1.27)))
-    )
-    (property "Value" "TBU-CA065-200-WH" (at 171.45 99.695 0)
-      (effects (font (size 1.27 1.27)))
-    )
-    (property "Footprint" "MACHADA_footprints:TBU-CA065-200-WH" (at 169.545 99.06 0)
-      (effects (font (size 1.27 1.27)) hide)
-    )
-    (property "Datasheet" "" (at 169.545 99.06 0)
-      (effects (font (size 1.27 1.27)) hide)
-    )
-    (pin "1")
-    (pin "2")
-    (instances
-      (project "Eco_display"
-        (path "/8b9448db-4b1d-4fc2-a488-03ccb6a18691/342f5a5a-4095-4f7f-8eba-841feace6be3"
-          (reference "U6") (unit 1)
-        )
-      )
-      (project "BIM_PCB"
-        (path "/b79ebed7-e146-448b-8dab-0aefb3e182ca/1465f310-1de3-424a-8f4a-a980ed628081"
-          (reference "U6") (unit 1)
-        )
-        (path "/b79ebed7-e146-448b-8dab-0aefb3e182ca/34e5006d-2f61-4d7d-acbf-5a24a5d8c7fc"
-          (reference "U12") (unit 1)
-        )
-        (path "/b79ebed7-e146-448b-8dab-0aefb3e182ca/2e21452f-cdd1-4ce6-a8e8-98e1abc18b72"
-          (reference "U20") (unit 1)
-        )
-      )
-      (project "MAX485"
-        (path "/bc82bdd3-8c90-4895-abd4-de755b621eab"
-          (reference "U16") (unit 1)
-        )
-      )
-      (project "ELIESTER_V2"
-        (path "/efe55700-0211-4481-aa01-7a7eb74def17/d62e2e8a-503b-4c7c-a2bb-b074e6b71fb0"
-          (reference "U16") (unit 1)
         )
       )
@@
         )
       )
+    )
+  )
+  (symbol (lib_id "Device:L") (at 170.815 87.63 90) (unit 1)
+    (in_bom yes) (on_board yes) (dnp no)
+    (property "Reference" "L1" (at 170.815 81.915 90)
+      (effects (font (size 1.27 1.27)))
+    )
+    (property "Value" "L" (at 170.815 84.455 90)
+      (effects (font (size 1.27 1.27)))
+    )
+    (property "Footprint" "Inductor_SMD:L_0402_1005Metric" (at 170.815 87.63 0)
+      (effects (font (size 1.27 1.27)) hide)
+    )
+    (property "Datasheet" "~" (at 170.815 87.63 0)
+      (effects (font (size 1.27 1.27)) hide)
+    )
+    (property "MPN" "BLM15HD182SN1D" (at 170.815 88.9 90)
+      (effects (font (size 1.27 1.27)))
+    )
+    (pin "1")
+    (pin "2")
+    (instances
+      (project "Eco_display"
+        (path "/8b9448db-4b1d-4fc2-a488-03ccb6a18691/342f5a5a-4095-4f7f-8eba-841feace6be3"
+          (reference "L1") (unit 1)
+        )
+      )
